File: Reflectance_Adapter/Reflectance_Adapter.kicad_sch (KiCad schematic)
At the start: 4 parts, among them J1 Reflector I2C, J2 Conn_QTRX_Top_Row, J3 Conn_QTRX_Bot_Row, U1 TCA9555PWR

Commit message: Assigned footprints
Parts:
- J2: footprint (none) -> Connector_PinSocket_2.54mm:PinSocket_1x08_P2.54mm_Vertical
- J3: footprint (none) -> Connector_PinSocket_2.54mm:PinSocket_1x11_P2.54mm_Vertical
Changed lines of the file:
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@@
 			)
 		)
-		(property "Footprint" ""
+		(property "Footprint" "Connector_PinSocket_2.54mm:PinSocket_1x11_P2.54mm_Vertical"
 			(at 246.38 90.17 0)
 			(effects
@@
 			)
 		)
-		(property "Footprint" ""
+		(property "Footprint" "Connector_PinSocket_2.54mm:PinSocket_1x08_P2.54mm_Vertical"
 			(at 222.25 90.17 0)
 			(effects

Commit message: Completed layout
User layer 1 contains dimensions of Pololu reflectance sensor array board. User layer 8 contains dimensions of slots of Pololu Chassis (copied over from the MSPM0 kicad project)
Parts:
- added J4: Support, Connector_PinHeader_2.54mm:PinHeader_1x04_P2.54mm_Vertical, symbol Connector:Conn_01x04_Pin
Connections:
- no-connect marks 1 -> 5
Changed lines of the file:
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@@
+	)
+	(no_connect
+		(at 85.09 118.11)
+	)
+	(no_connect
+		(at 85.09 120.65)
 	)
 	(no_connect
 		(at 143.51 81.28)
+	)
+	(no_connect
+		(at 85.09 123.19)
+	)
+	(no_connect
+		(at 85.09 115.57)
 	)
 	(wire
@@
 					(unit 1)
 				)
+			)
+		)
+	)
+	(symbol
+		(lib_name "Conn_01x04_Pin_1")
+		(lib_id "Connector:Conn_01x04_Pin")
+		(at 80.01 118.11 0)
+		(unit 1)
+		(exclude_from_sim no)
+		(in_bom yes)
+		(on_board yes)
+		(dnp no)
+		(property "Reference" "J4"
+			(at 77.978 111.252 0)
+			(effects
+				(font
+					(size 1.27 1.27)
+				)
+			)
+		)
+		(property "Value" "Support"
+			(at 78.232 113.538 0)
+			(effects
+				(font
+					(size 1.27 1.27)
+				)
+			)
+		)
+		(property "Footprint" "Connector_PinHeader_2.54mm:PinHeader_1x04_P2.54mm_Vertical"
+			(at 85.344 125.476 0)
+			(effects
+				(font
+					(size 1.27 1.27)
+				)
+				(hide yes)
+			)
+		)
+		(property "Datasheet" "~"
+			(at 80.01 118.11 0)
+			(effects
+				(font
+					(size 1.27 1.27)
+				)
+				(hide yes)
+			)
+		)
+		(property "Description" "Generic connector, single row, 01x04, script generated"
+			(at 86.36 128.778 0)
+			(effects
+				(font
+					(size 1.27 1.27)
+				)
+				(hide yes)
+			)
+		)
+		(pin "4"
+		)
+		(pin "3"
+		)
+		(pin "2"
+		)
+		(pin "1"
+		)
+		(instances
+			(project "Reflectance_Adapter"
+				(path "/52ddd7c2-7a01-4e6e-b0f5-c4fe3dfba013"
+					(reference "J4")
+					(unit 1)
+				)

Commit message: corrected i2c pin positions
Connections:
- net SCL: now also J1.4 (Pin_4); no longer J1.3 (Pin_3)
- net SDA: now also J1.3 (Pin_3); no longer J1.4 (Pin_4)
Changed lines of the file:
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@@
 		)
 	)
-	(label "SCL"
+	(label "SDA"
 		(at 119.38 77.47 0)
 		(fields_autoplaced yes)
@@
 		)
 	)
-	(label "SDA"
+	(label "SCL"
 		(at 119.38 80.01 0)
 		(fields_autoplaced yes)
